Commit message: Add XgoDuck roller model and Swizzle task
Add the SolidWorks-aligned four-wheel roller model and adapt the MicroDuck
Swizzle recipe for XgoDuck. Keep both skates grounded, hold the head at its
default posture, and use progressive bearing-drag and heading curricula.

Align shared CAD inertials, HLS1910 retest parameters, and actuator timing.
Update Walk foot-lift, backward-practice, and head-command curricula. Fix
servo-only ONNX metadata and document roller training and playback. Use
standard PyPI lock sources without changing dependency versions.

Validation: 215 tests passed, 1 skipped. The Swizzle smoke test completed
5 iterations with 64 environments; ONNX inference and 61-input/14-output
metadata checks passed.

File: src/mjlab_microduck/robot/xgoduck/urdf/XGODUCK.urdf (robot description, URDF)
Before this commit: robot xgoduck_v2, 15 links, 14 joints
Links:
- link head_pitch: mass 0.0042717593 -> 0.004004831969378556
- link head_roll: mass 0.16746559 -> 0.1743404125948065
- link head_yaw: mass 0.035199775 -> 0.03582857464025031
- link left_ankle: mass 0.030933135 -> 0.02928955584072766
- link left_hip_pitch: mass 0.056532972 -> 0.05875913250549258
- link left_hip_roll: mass 0.010666598 -> 0.009655706396208049
- link left_hip_yaw: mass 0.030933135 -> 0.03170602779137935
- link left_knee: mass 0.026666496 -> 0.02471174850017473
- link neck_pitch: mass 0.043733053 -> 0.04674973451754257
- link right_ankle: mass 0.030933135 -> 0.02928955071377668
- link right_hip_pitch: mass 0.056532972 -> 0.05875913339225547
- link right_hip_roll: mass 0.010666598 -> 0.009655706396208049
- link right_hip_yaw: mass 0.030933135 -> 0.03170602779137936
- link right_knee: mass 0.026666496 -> 0.02471174850017473
- link trunk_base: mass 0.23786514 -> 0.2286207806414798
